Commit message: Activities for learning about UUV Simulator

File: bluerov2_description/urdf/snippets.xacro (robot description, xacro)
@@ -101,3 +101,64 @@
     </xacro:regular_camera_plugin_macro>
   </xacro:macro>
+  <xacro:macro name="bluerov_altimeter"
+    params="namespace suffix parent_link topic mass update_rate
+      samples fov *origin">
+    <!-- Sensor link -->
+    <link name="${namespace}/altimeter${suffix}_link">
+      <inertial>
+        <inertia ixx="0.00001" ixy="0.0" ixz="0.0" iyy="0.00001" iyz="0.0" izz="0.00001" />
+        <mass value="${mass}" />
+        <origin xyz="0 0 0" rpy="0 0 0" />
+      </inertial>
+      <visual>
+        <geometry>
+          <mesh filename="file://$(find uuv_sensor_ros_plugins)/meshes/oe14-372.dae" scale="1 1 1"/>
+        </geometry>
+      </visual>
+      <xacro:no_collision/>
+    </link>
+    <joint name="${namespace}_altimeter${suffix}_joint" type="revolute">
+      <xacro:insert_block name="origin" />
+      <parent link="${parent_link}" />
+      <child link="${namespace}/altimeter${suffix}_link" />
+      <limit upper="0" lower="0" effort="0" velocity="0" />
+      <axis xyz="1 0 0"/>
+    </joint>
+    <gazebo reference="${namespace}/altimeter${suffix}_link">
+      <sensor type="ray" name="sonar">
+          <pose>0.25 0 0 0 0 0</pose>
+          <update_rate>"${update_rate}"</update_rate>
+          <ray>
+            <scan>
+              <horizontal>
+                <samples>"${samples}"</samples>
+                <resolution>1.0</resolution>
+                <min_angle>-0.25</min_angle>
+                <max_angle>0.25</max_angle>
+              </horizontal>
+              <vertical>
+                <samples>"${samples}"</samples>
+                <resolution>1</resolution>
+                <min_angle>-0.25</min_angle>
+                <max_angle>0.25</max_angle>
+              </vertical>
+            </scan>
+            <range>
+              <min>0.01</min>
+              <max>30.0</max>
+              <resolution>0.001</resolution>
+            </range>
+          </ray>
+          <plugin filename="libgazebo_ros_range.so" name="gazebo_ros_range">
+            <gaussianNoise>0.005</gaussianNoise>
+            <alwaysOn>true</alwaysOn>
+            <updateRate>"${update_rate}"</updateRate>
+            <topicName>"${topic}"</topicName>
+            <frameName>"altimeter${suffix}_link"</frameName>
+            <fov>"${fov}"</fov>
+            <radiation>ultrasound</radiation>
+          </plugin>
+        </sensor>
+    </gazebo>
+  </xacro:macro>
 </robot>
