Commit message: Overhaul to combine Ardusub SITL and Gazebo 9

File: bluerov2_description/urdf/base.xacro (robot description, xacro)
@@ -13,5 +13,5 @@
   -->
   <!-- Mass -->
-  <xacro:property name="mass" value="10"/>
+  <xacro:property name="mass" value="11.2"/>
   <!-- Describing the dimensions of the vehicle's bounding box: width, length, height -->
   <xacro:property name="x_size" value="0.448"/>

File: bluerov2_description/urdf/sensors.xacro (robot description, xacro)
@@ -17,13 +17,7 @@
     <origin xyz="0 0 0" rpy="0 0 0"/>
   </xacro:default_pressure>
-  <!-- Beacon Sensor  -->
-  <!--
-  <xacro:default_beacon namespace="${namespace}" parent_link="${namespace}/base_link">
-    <origin xyz="0 0 0" rpy="0 0 0"/>
-  </xacro:default_beacon>
--->
   <!-- Mount a camera -->
-  <!-- <xacro:default_camera namespace="${namespace}" parent_link="${namespace}/base_link" suffix="front">
-    <origin xyz="0 0 0.2" rpy="0 0 0"/>
-  </xacro:default_camera> -->
+  <xacro:bluerov_camera namespace="" parent_link="${namespace}/base_link" suffix="_front">
+    <origin xyz="0.2 0 0" rpy="0 0 0"/>
+  </xacro:bluerov_camera>
 </robot>

File: bluerov2_description/urdf/snippets.xacro (robot description, xacro)
@@ -84,3 +84,20 @@
     </gazebo>
   </xacro:macro>
+  <xacro:macro name="bluerov_camera" params="namespace parent_link suffix *origin">
+    <xacro:regular_camera_plugin_macro
+      namespace="${namespace}"
+      suffix="${suffix}"
+      parent_link="${parent_link}"
+      topic="camera"
+      mass="0.001"
+      update_rate="30"
+      hfov="1.5125"
+      width="1920"
+      height="1080"
+      stddev="0.01"
+      scale="1.0">
+      <inertia ixx="0.00001" ixy="0.0" ixz="0.0" iyy="0.00001" iyz="0.0" izz="0.00001" />
+      <xacro:insert_block name="origin" />
+    </xacro:regular_camera_plugin_macro>
+  </xacro:macro>
 </robot>

Commit message: Robot configuration for ping1d altimeter added

File: bluerov2_description/urdf/base.xacro (robot description, xacro)
@@ -72,10 +72,10 @@
         </visual>
         <!-- In rexrov2_base they made collision planes to minize the GPU load -->
-        <!-- <collision>
+        <collision>
           <origin xyz="0 0 0" rpy="0 0 0"/>
           <geometry>
             <mesh filename="${collision_mesh_file}" scale="1 1 1" />
           </geometry>
-        </collision> -->
+        </collision>
       </link>
     <gazebo reference="${namespace}/base_link">

File: bluerov2_description/urdf/snippets.xacro (robot description, xacro)
@@ -102,17 +102,17 @@
   </xacro:macro>
   <xacro:macro name="bluerov_altimeter"
-    params="namespace suffix parent_link topic mass update_rate
-      samples fov *origin">
+    params="namespace suffix parent_link *origin">
     <!-- Sensor link -->
     <link name="${namespace}/altimeter${suffix}_link">
       <inertial>
         <inertia ixx="0.00001" ixy="0.0" ixz="0.0" iyy="0.00001" iyz="0.0" izz="0.00001" />
-        <mass value="${mass}" />
-        <origin xyz="0 0 0" rpy="0 0 0" />
+        <mass value="0.01" />
+        <origin xyz="0 0 0" rpy="0 0 0"/>
       </inertial>
       <visual>
         <geometry>
-          <mesh filename="file://$(find uuv_sensor_ros_plugins)/meshes/oe14-372.dae" scale="1 1 1"/>
+          <mesh filename="file://$(find bluerov2_description)/meshes/ping1d.dae" scale="1 1 1"/>
         </geometry>
+        <origin xyz="0 0 0" rpy="0 0 -${0.5*pi}"/>
       </visual>
       <xacro:no_collision/>
@@ -127,19 +127,19 @@
     <gazebo reference="${namespace}/altimeter${suffix}_link">
       <sensor type="ray" name="sonar">
-          <pose>0.25 0 0 0 0 0</pose>
-          <update_rate>"${update_rate}"</update_rate>
+          <pose>0 0 0 0 0 0</pose>
+          <update_rate>15.0</update_rate>
           <ray>
             <scan>
               <horizontal>
-                <samples>"${samples}"</samples>
-                <resolution>1.0</resolution>
-                <min_angle>-0.25</min_angle>
-                <max_angle>0.25</max_angle>
+                <samples>5.0</samples>
+                <resolution>1</resolution>
+                <min_angle>-${15*pi/180}</min_angle>
+                <max_angle>${15*pi/180}</max_angle>
               </horizontal>
               <vertical>
-                <samples>"${samples}"</samples>
+                <samples>5.0</samples>
                 <resolution>1</resolution>
-                <min_angle>-0.25</min_angle>
-                <max_angle>0.25</max_angle>
+                <min_angle>-${15*pi/180}</min_angle>
+                <max_angle>${15*pi/180}</max_angle>
               </vertical>
             </scan>
@@ -153,8 +153,8 @@
             <gaussianNoise>0.005</gaussianNoise>
             <alwaysOn>true</alwaysOn>
-            <updateRate>"${update_rate}"</updateRate>
-            <topicName>"${topic}"</topicName>
-            <frameName>"altimeter${suffix}_link"</frameName>
-            <fov>"${fov}"</fov>
+            <updateRate>15.0</updateRate>
+            <topicName>altimeter${suffix}</topicName>
+            <frameName>${namespace}/altimeter${suffix}_link</frameName>
+            <fov>${30*pi/180}</fov>
             <radiation>ultrasound</radiation>
           </plugin>

Commit message: Packages prepared to work with neptus playground and IMC bridge

File: bluerov2_description/urdf/base.xacro (robot description, xacro)
@@ -28,5 +28,5 @@
   assume NWU (otherwise cob is below cog?). 0.155
   -->
-  <xacro:property name="cob" value="0 0 0"/>
+  <xacro:property name="cob" value="0 0 0.3872"/>
   <!-- Fluid density -->
   <xacro:property name="rho" value="1028"/>

File: bluerov2_description/urdf/sensors.xacro (robot description, xacro)
@@ -21,3 +21,5 @@
     <origin xyz="0.2 0 0" rpy="0 0 0"/>
   </xacro:bluerov_camera>
+  <!-- Mount a GPS. -->
+  <xacro:default_gps namespace="${namespace}" parent_link="${namespace}/base_link" />
 </robot>
